File: dc5v-for-atari-stf.kicad_sch (KiCad schematic)
At the start: 13 parts, among them J1 Conn_01x03, J2 Conn_01x06, J3 Adjustable MT3608 module, J4 Fixed 12V module, J5 Conn_01x02, SW1 Momentary or Latched

Commit message: tweak labels
Other:
- title: DC5V for the Atari STF -> DC5V for the Atari STf/e/...
Changed lines of the file:
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@@
   (paper "A4" portrait)
   (title_block
-    (title "DC5V for the Atari STF")
+    (title "DC5V for the Atari STf/e/...")
     (date "2023-08-24")
     (rev "v1.0.0-RC1")
